File: 19. ESP32 Module.kicad_pcb (KiCad board)
At the start: 2 copper layers, 40 x 60 mm, 63 parts, among them J1 Conn_01x14_Pin, J2 Conn_01x14_Pin, J3 USB_C_Receptacle_USB2.0_16P, J4 INPUT, J5 POWER, SW1 K1, SW2 K2, SW3 K1, U1 ESP32-S3, U2 W25Q128JVS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

Commit message: Initial commit
Routing:
- added copper zone on In1.Cu, net GND
- added copper zone on In2.Cu, net GND
Other:
- copper layers 2 -> 4
Changed lines of the file:
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@@
 	(layers
 		(0 "F.Cu" signal)
+		(1 "In1.Cu" signal)
+		(2 "In2.Cu" signal)
 		(31 "B.Cu" signal)
 		(32 "B.Adhes" user "B.Adhesive")
@@
 			)
 			(layer "dielectric 1"
+				(type "prepreg")
+				(thickness 0.1)
+				(material "FR4")
+				(epsilon_r 4.5)
+				(loss_tangent 0.02)
+			)
+			(layer "In1.Cu"
+				(type "copper")
+				(thickness 0.035)
+			)
+			(layer "dielectric 2"
 				(type "core")
-				(thickness 1.51)
+				(thickness 1.24)
+				(material "FR4")
+				(epsilon_r 4.5)
+				(loss_tangent 0.02)
+			)
+			(layer "In2.Cu"
+				(type "copper")
+				(thickness 0.035)
+			)
+			(layer "dielectric 3"
+				(type "prepreg")
+				(thickness 0.1)
 				(material "FR4")
 				(epsilon_r 4.5)
@@
 	)
 	(zone
-		(net 3)
-		(net_name "+3.3V")
-		(layers "F&B.Cu")
+		(net 1)
+		(net_name "GND")
+		(layers "F.Cu" "In1.Cu" "In2.Cu" "B.Cu")
 		(hatch edge 0.5)
-		(priority 3)
 		(connect_pads yes
 			(clearance 0.5)
@@
 		(polygon
 			(pts
-				(xy 147.53 51.98) (xy 146 51.98) (xy 145.46 52.52) (xy 144.74 52.52) (xy 144.74 51.32) (xy 147.53 51.32)
+				(xy 175.7 39.17) (xy 134.52 39.17) (xy 134.52 96.87) (xy 136.35 98.7) (xy 174.05 98.7) (xy 175.7 97.05)
 			)
 		)
@@
 		(polygon
 			(pts
-				(xy 154.9 49.58) (xy 157.46 49.58) (xy 157.46 45.38) (xy 157.43 45.35) (xy 155.66 45.35) (xy 155.2 45.81)
-				(xy 155.2 48.66) (xy 155.2 48.659882) (xy 154.9 48.97)
+				(xy 147.53 51.98) (xy 146 51.98) (xy 145.46 52.52) (xy 144.74 52.52) (xy 144.74 51.32) (xy 147.53 51.32)
 			)
 		)
 	)
 	(zone
-		(net 1)
-		(net_name "GND")
+		(net 3)
+		(net_name "+3.3V")
 		(layers "F&B.Cu")
 		(hatch edge 0.5)
+		(priority 3)
 		(connect_pads yes
 			(clearance 0.5)
@@
 		(polygon
 			(pts
-				(xy 175.7 39.17) (xy 134.52 39.17) (xy 134.52 96.87) (xy 136.35 98.7) (xy 174.05 98.7) (xy 175.7 97.05)
+				(xy 154.9 49.58) (xy 157.46 49.58) (xy 157.46 45.38) (xy 157.43 45.35) (xy 155.66 45.35) (xy 155.2 45.81)
+				(xy 155.2 48.66) (xy 155.2 48.659882) (xy 154.9 48.97)
 			)
 		)
